File: pcb/_autosave-bd64pcb.sch (KiCad schematic (older format))
At the start: 239 parts, among them J1 USB_C_Receptacle_USB2.0, J2 USB_B_Micro, SW1 SW_Push, U1 ATmega32U4-MU, U2 MCP23017_ML, U3 IS31FL3733-QF, Y1 16MHz

Commit message: no good traces yet
Parts:
- MX1, MX2, MX3: footprint MX_Alps_Hybrid:MX-1U-NoLED -> MX_Only:MXOnly-1U-NoLED
Changed lines of the file:
@@
 F 0 "MX3" H 10450 2225 60  0000 C CNN
 F 1 "MX-NoLED" H 10450 2150 20  0000 C CNN
-F 2 "MX_Alps_Hybrid:MX-1U-NoLED" H 9850 2000 60  0001 C CNN
+F 2 "MX_Only:MXOnly-1U-NoLED" H 9850 2000 60  0001 C CNN
 F 3 "" H 9850 2000 60  0001 C CNN
 	1    10475 2025
@@
 F 0 "MX2" H 9825 2225 60  0000 C CNN
 F 1 "MX-NoLED" H 9825 2150 20  0000 C CNN
-F 2 "MX_Alps_Hybrid:MX-1U-NoLED" H 9225 2000 60  0001 C CNN
+F 2 "MX_Only:MXOnly-1U-NoLED" H 9225 2000 60  0001 C CNN
 F 3 "" H 9225 2000 60  0001 C CNN
 	1    9850 2025
@@
 F 0 "MX1" H 9200 2225 60  0000 C CNN
 F 1 "MX-NoLED" H 9200 2150 20  0000 C CNN
-F 2 "MX_Alps_Hybrid:MX-1U-NoLED" H 8600 2000 60  0001 C CNN
+F 2 "MX_Only:MXOnly-1U-NoLED" H 8600 2000 60  0001 C CNN
 F 3 "" H 8600 2000 60  0001 C CNN
 	1    9225 2025
