File: pcb/_autosave-bd64pcb.kicad_pcb (KiCad board)
At the start: 2 copper layers, 266.7 x 95.2 mm, 245 parts, among them J1 USB_C_Receptacle_USB2.0, SW1 SW_Push, U1 ATmega32U4-MU, U2 MCP23017_ML, U3 IS31FL3733-QF, Y1 16MHz

Commit message: gitignore
Routing:
- net SW3: track 342.3 -> 345.1 mm
- net SW1: track 322.1 -> 323.5 mm
