File: pcb/bd64pcb.kicad_sch (KiCad schematic)
At the start: 227 parts, among them J1 USB_C_Receptacle_USB2.0, J2 Conn_01x04, J3 Conn_01x04, SW1 SW_Push, U1 ATmega32U4-MU, U2 IS31FL3733-QF, Y1 16MHz

Commit message: add Ω to sch values
Parts:
- R1, R2: value 5.1k -> 5.1kΩ
- R10, R11: value 100k -> 100kΩ
- R12: value 20k -> 20kΩ
- R3, R9: value 10k -> 10kΩ
- R4, R8: value 22 -> 22Ω
- R5, R6, R7: value 4.7k -> 4.7kΩ
Changed lines of the file:
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@@
     (in_bom yes) (on_board yes)
     (property "Reference" "R9" (id 0) (at 128.905 92.075 90))
-    (property "Value" "10k" (id 1) (at 128.905 93.98 90)
+    (property "Value" "10kΩ" (id 1) (at 128.905 93.98 90)
       (effects (font (size 0.9906 0.9906)))
     )
@@
     (in_bom yes) (on_board yes)
     (property "Reference" "R4" (id 0) (at 83.82 64.135 90))
-    (property "Value" "22" (id 1) (at 83.82 66.04 90)
+    (property "Value" "22Ω" (id 1) (at 83.82 66.04 90)
       (effects (font (size 0.9906 0.9906)))
     )
@@
     (in_bom yes) (on_board yes)
     (property "Reference" "R8" (id 0) (at 83.82 70.485 90))
-    (property "Value" "22" (id 1) (at 83.82 68.58 90)
+    (property "Value" "22Ω" (id 1) (at 83.82 68.58 90)
       (effects (font (size 0.9906 0.9906)))
     )
@@
     (in_bom yes) (on_board yes)
     (property "Reference" "R3" (id 0) (at 89.535 36.83 90))
-    (property "Value" "10k" (id 1) (at 91.5416 36.83 90)
+    (property "Value" "10kΩ" (id 1) (at 91.5416 36.83 90)
       (effects (font (size 0.9906 0.9906)))
     )
@@
       (effects (font (size 1.27 1.27)) (justify left))
     )
-    (property "Value" "20k" (id 1) (at 40.005 205.105 90)
+    (property "Value" "20kΩ" (id 1) (at 40.005 205.105 90)
       (effects (font (size 0.9906 0.9906)) (justify left))
     )
@@
     (in_bom yes) (on_board yes)
     (property "Reference" "R2" (id 0) (at 52.07 83.82 90))
-    (property "Value" "5.1k" (id 1) (at 52.07 82.0166 90)
+    (property "Value" "5.1kΩ" (id 1) (at 52.07 82.0166 90)
       (effects (font (size 0.9906 0.9906)))
     )
@@
     (in_bom yes) (on_board yes)
     (property "Reference" "R1" (id 0) (at 52.07 76.2 90))
-    (property "Value" "5.1k" (id 1) (at 52.07 78.105 90)
+    (property "Value" "5.1kΩ" (id 1) (at 52.07 78.105 90)
       (effects (font (size 0.9906 0.9906)))
     )
@@
       (effects (font (size 1.27 1.27)) (justify left))
     )
-    (property "Value" "100k" (id 1) (at 45.085 198.755 90)
+    (property "Value" "100kΩ" (id 1) (at 45.085 198.755 90)
       (effects (font (size 0.9906 0.9906)) (justify left))
     )
@@
       (effects (font (size 1.27 1.27)) (justify left))
     )
-    (property "Value" "100k" (id 1) (at 40.005 198.755 90)
+    (property "Value" "100kΩ" (id 1) (at 40.005 198.755 90)
       (effects (font (size 0.9906 0.9906)) (justify left))
     )
@@
     (in_bom yes) (on_board yes)
     (property "Reference" "R5" (id 0) (at 131.445 66.675 90))
-    (property "Value" "4.7k" (id 1) (at 133.35 66.675 90)
+    (property "Value" "4.7kΩ" (id 1) (at 133.35 66.675 90)
       (effects (font (size 0.9906 0.9906)))
     )
@@
     (in_bom yes) (on_board yes)
     (property "Reference" "R6" (id 0) (at 135.255 66.675 90))
-    (property "Value" "4.7k" (id 1) (at 137.16 66.675 90)
+    (property "Value" "4.7kΩ" (id 1) (at 137.16 66.675 90)
       (effects (font (size 0.9906 0.9906)))
     )
@@
     (in_bom yes) (on_board yes)
     (property "Reference" "R7" (id 0) (at 139.065 66.675 90))
-    (property "Value" "4.7k" (id 1) (at 140.97 66.675 90)
+    (property "Value" "4.7kΩ" (id 1) (at 140.97 66.675 90)
       (effects (font (size 0.9906 0.9906)))
     )
@@
     )
     (path "/00000000-0000-0000-0000-00006c136ea4"
-      (reference "R1") (unit 1) (value "5.1k") (footprint "Resistor_SMD:R_0805_2012Metric")
+      (reference "R1") (unit 1) (value "5.1kΩ") (footprint "Resistor_SMD:R_0805_2012Metric")
     )
     (path "/00000000-0000-0000-0000-00006c136e9e"
-      (reference "R2") (unit 1) (value "5.1k") (footprint "Resistor_SMD:R_0805_2012Metric")
+      (reference "R2") (unit 1) (value "5.1kΩ") (footprint "Resistor_SMD:R_0805_2012Metric")
     )
     (path "/00000000-0000-0000-0000-0000629b7d20"
-      (reference "R3") (unit 1) (value "10k") (footprint "Resistor_SMD:R_0805_2012Metric")
+      (reference "R3") (unit 1) (value "10kΩ") (footprint "Resistor_SMD:R_0805_2012Metric")
     )
     (path "/00000000-0000-0000-0000-000062962336"
-      (reference "R4") (unit 1) (value "22") (footprint "Resistor_SMD:R_0805_2012Metric")
+      (reference "R4") (unit 1) (value "22Ω") (footprint "Resistor_SMD:R_0805_2012Metric")
     )
     (path "/00000000-0000-0000-0000-0000841aa3ed"
-      (reference "R5") (unit 1) (value "4.7k") (footprint "Resistor_SMD:R_0805_2012Metric")
+      (reference "R5") (unit 1) (value "4.7kΩ") (footprint "Resistor_SMD:R_0805_2012Metric")
     )
     (path "/00000000-0000-0000-0000-00008429a964"
-      (reference "R6") (unit 1) (value "4.7k") (footprint "Resistor_SMD:R_0805_2012Metric")
+      (reference "R6") (unit 1) (value "4.7kΩ") (footprint "Resistor_SMD:R_0805_2012Metric")
     )
     (path "/00000000-0000-0000-0000-00008429af53"
-      (reference "R7") (unit 1) (value "4.7k") (footprint "Resistor_SMD:R_0805_2012Metric")
+      (reference "R7") (unit 1) (value "4.7kΩ") (footprint "Resistor_SMD:R_0805_2012Metric")
     )
     (path "/00000000-0000-0000-0000-000062962ab2"
-      (reference "R8") (unit 1) (value "22") (footprint "Resistor_SMD:R_0805_2012Metric")
+      (reference "R8") (unit 1) (value "22Ω") (footprint "Resistor_SMD:R_0805_2012Metric")
     )
     (path "/00000000-0000-0000-0000-00006295dcd9"
-      (reference "R9") (unit 1) (value "10k") (footprint "Resistor_SMD:R_0805_2012Metric")
+      (reference "R9") (unit 1) (value "10kΩ") (footprint "Resistor_SMD:R_0805_2012Metric")
     )
     (path "/00000000-0000-0000-0000-00007b0aaa9f"
-      (reference "R10") (unit 1) (value "100k") (footprint "Resistor_SMD:R_0805_2012Metric")
+      (reference "R10") (unit 1) (value "100kΩ") (footprint "Resistor_SMD:R_0805_2012Metric")
     )
     (path "/00000000-0000-0000-0000-00007a98bff2"
-      (reference "R11") (unit 1) (value "100k") (footprint "Resistor_SMD:R_0805_2012Metric")
+      (reference "R11") (unit 1) (value "100kΩ") (footprint "Resistor_SMD:R_0805_2012Metric")
     )
     (path "/00000000-0000-0000-0000-0000693557b1"
-      (reference "R12") (unit 1) (value "20k") (footprint "Resistor_SMD:R_0805_2012Metric")
+      (reference "R12") (unit 1) (value "20kΩ") (footprint "Resistor_SMD:R_0805_2012Metric")
     )
     (path "/00000000-0000-0000-0000-0000629b57e0"

Commit message: usbc removed; surrogate jst connected
Parts:
- removed F1: 500mA, Fuse:Fuse_1206_3216Metric, symbol Device:Polyfuse_Small
- removed J1: USB_C_Receptacle_USB2.0, Connector_USB:USB_C_Receptacle_HRO_TYPE-C-31-M-12, symbol Connector:USB_C_Receptacle_USB2.0
- removed R1, R2: 5.1kΩ, Resistor_SMD:R_0805_2012Metric, symbol Device:R_Small
- added J1: Conn_01x04, Connector_JST:JST_SUR_SM04B-SURS-TF_1x04-1MP_P0.80mm_Horizontal, symbol Connector_Generic:Conn_01x04
Connections:
- net +5V: now also J1.1 (Pin_1)
- net D+: now also J1.3 (Pin_3)
- net D-: now also J1.2 (Pin_2)
- net GND: now also J1.4 (Pin_4), J1.MP
- no-connect marks 3 -> 1
