File: pcb/usbc_daughterboard/usbc64/usbc64.kicad_sch (KiCad schematic)
At the start: 5 parts, among them J1 USB_C_Receptacle_USB2.0

Commit message: sch and pcb rough starts
Parts:
- removed R?: R_Small, symbol Device:R_Small
- added F1: 500mA, symbol Device:Polyfuse_Small
- added H1: MountingHole_Pad, symbol Mechanical:MountingHole_Pad
- added H2, H3, H4: MountingHole, symbol Mechanical:MountingHole
- added R1, R2: 5.1kΩ, Resistor_SMD:R_0805_2012Metric, symbol Device:R_Small
- J2: renamed from J?; footprint (none) -> Connector_JST:JST_SUR_SM04B-SURS-TF_1x04-1MP_P0.80mm_Horizontal
- L1: renamed from L?; value L_Ferrite -> 60R@100MHz; footprint (none) -> Inductor_SMD:L_1206_3216Metric; symbol Device:L_Ferrite -> Device:L_Ferrite_Small
- gave numbers to parts that had none: 1
Connections:
- net GND: now reaches L1.1
- net GND: now also J2.MP
- net +5V: now reaches L1.2
- net +5V: now also J1.A1 (GND), J1.A12 (GND), J1.B1 (GND), J1.B12 (GND), J1.S1 (SHIELD), U1.3 (GND), U1.8 (GND), F1.2, H1.1, R1.2, R2.1
- net VBUS: now reaches J1.A4 (VBUS), J1.A9 (VBUS), J1.B4 (VBUS), J1.B9 (VBUS)
- net VBUS: now also F1.1
- net at J1.A5 (CC1): now also R1.1
- net at J1.B5 (CC2): now also R2.2
- no-connect marks 0 -> 2
Other:
- moved on the sheet: J1, J2, U1

Commit message: mounting holes
Parts:
- H1, H2, H3, H4: footprint (none) -> MountingHole:MountingHole_2.2mm_M2_Pad
Connections:
- net +5V: no longer H1.1, J1.A1 (GND), J1.A12 (GND), J1.B1 (GND), J1.B12 (GND), J1.S1 (SHIELD), L1.2, R1.2, R2.1, U1.3 (GND), U1.8 (GND)
- new net GNDPWR: H1.1, J1.A1 (GND), J1.A12 (GND), J1.B1 (GND), J1.B12 (GND), J1.S1 (SHIELD), L1.2, R1.2, R2.1, U1.3 (GND), U1.8 (GND)
Changed lines of the file:
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@@
 (kicad_sch (version 20211123) (generator eeschema)
   (paper "A5")
-  (junction (at 96.52 43.18) (diameter 0) (color 0 0 0 0)
-  )
   (junction (at 73.66 50.165) (diameter 0) (color 0 0 0 0)
   )
@@
     (stroke (width 0) (type default) (color 0 0 0 0))
   )
-  (wire (pts (xy 96.52 43.18) (xy 96.52 44.45))
-    (stroke (width 0) (type default) (color 0 0 0 0))
-  )
   (wire (pts (xy 88.9 73.025) (xy 88.9 71.755))
     (stroke (width 0) (type default) (color 0 0 0 0))
@@
     (stroke (width 0) (type default) (color 0 0 0 0))
   )
-  (wire (pts (xy 96.52 43.18) (xy 97.79 43.18))
-    (stroke (width 0) (type default) (color 0 0 0 0))
-  )
   (wire (pts (xy 95.25 71.755) (xy 96.52 71.755))
     (stroke (width 0) (type default) (color 0 0 0 0))
@@
     (stroke (width 0) (type default) (color 0 0 0 0))
   )
-  (wire (pts (xy 93.98 43.18) (xy 96.52 43.18))
+  (wire (pts (xy 93.98 43.18) (xy 97.79 43.18))
     (stroke (width 0) (type default) (color 0 0 0 0))
   )
@@
   (symbol (lib_id "power:GNDPWR") (at 96.52 73.025 0) (unit 1)
     (in_bom yes) (on_board yes)
-    (property "Reference" "#PWR?" (id 0) (at 96.52 78.105 0)
+    (property "Reference" "#PWR0112" (id 0) (at 96.52 78.105 0)
       (effects (font (size 1.27 1.27)) hide)
     )
@@
       (effects (font (size 1.27 1.27)) (justify left))
     )
-    (property "Footprint" "" (id 2) (at 144.145 77.47 0)
+    (property "Footprint" "MountingHole:MountingHole_2.2mm_M2_Pad" (id 2) (at 144.145 77.47 0)
       (effects (font (size 1.27 1.27)) hide)
     )
@@
       (effects (font (size 1.27 1.27)) (justify left))
     )
-    (property "Footprint" "" (id 2) (at 142.875 62.23 0)
+    (property "Footprint" "MountingHole:MountingHole_2.2mm_M2_Pad" (id 2) (at 142.875 62.23 0)
       (effects (font (size 1.27 1.27)) hide)
     )
@@
   (symbol (lib_id "power:GNDPWR") (at 73.66 50.165 0) (unit 1)
     (in_bom yes) (on_board yes)
-    (property "Reference" "#PWR?" (id 0) (at 73.66 55.245 0)
+    (property "Reference" "#PWR0107" (id 0) (at 73.66 55.245 0)
       (effects (font (size 1.27 1.27)) hide)
     )
@@
   (symbol (lib_id "power:GNDPWR") (at 48.895 81.915 0) (unit 1)
     (in_bom yes) (on_board yes)
-    (property "Reference" "#PWR?" (id 0) (at 48.895 86.995 0)
+    (property "Reference" "#PWR0106" (id 0) (at 48.895 86.995 0)
       (effects (font (size 1.27 1.27)) hide)
     )
@@
   (symbol (lib_id "power:GND") (at 88.9 73.025 0) (unit 1)
     (in_bom yes) (on_board yes)
-    (property "Reference" "#PWR?" (id 0) (at 88.9 79.375 0)
+    (property "Reference" "#PWR0108" (id 0) (at 88.9 79.375 0)
       (effects (font (size 1.27 1.27)) hide)
     )
@@
   (symbol (lib_id "power:GNDPWR") (at 139.065 63.5 0) (unit 1)
     (in_bom yes) (on_board yes)
-    (property "Reference" "#PWR?" (id 0) (at 139.065 68.58 0)
+    (property "Reference" "#PWR0114" (id 0) (at 139.065 68.58 0)
       (effects (font (size 1.27 1.27)) hide)
     )
@@
       (effects (font (size 1.27 1.27)) (justify left))
     )
-    (property "Footprint" "" (id 2) (at 144.145 72.39 0)
+    (property "Footprint" "MountingHole:MountingHole_2.2mm_M2_Pad" (id 2) (at 144.145 72.39 0)
       (effects (font (size 1.27 1.27)) hide)
     )
@@
   (symbol (lib_id "power:GNDPWR") (at 41.275 81.915 0) (unit 1)
     (in_bom yes) (on_board yes)
-    (property "Reference" "#PWR?" (id 0) (at 41.275 86.995 0)
+    (property "Reference" "#PWR0105" (id 0) (at 41.275 86.995 0)
       (effects (font (size 1.27 1.27)) hide)
     )
@@
   (symbol (lib_id "power:GNDPWR") (at 115.57 71.12 0) (unit 1)
     (in_bom yes) (on_board yes)
-    (property "Reference" "#PWR?" (id 0) (at 115.57 76.2 0)
+    (property "Reference" "#PWR0113" (id 0) (at 115.57 76.2 0)
       (effects (font (size 1.27 1.27)) hide)
     )
@@
       (effects (font (size 1.27 1.27)) (justify left))
     )
-    (property "Footprint" "" (id 2) (at 144.145 67.31 0)
+    (property "Footprint" "MountingHole:MountingHole_2.2mm_M2_Pad" (id 2) (at 144.145 67.31 0)
       (effects (font (size 1.27 1.27)) hide)
     )
@@
     )
   )
-  (symbol (lib_id "power:GNDPWR") (at 96.52 44.45 0) (unit 1)
-    (in_bom yes) (on_board yes)
-    (property "Reference" "#PWR?" (id 0) (at 96.52 49.53 0)
-      (effects (font (size 1.27 1.27)) hide)
-    )
-    (property "Value" "GNDPWR" (id 1) (at 96.52 46.99 0)
-      (effects (font (size 0.381 0.381)))
-    )
-    (property "Footprint" "" (id 2) (at 96.52 45.72 0)
-      (effects (font (size 1.27 1.27)) hide)
-    )
-    (property "Datasheet" "" (id 3) (at 96.52 45.72 0)
+  (symbol (lib_id "power:GNDPWR") (at 96.52 50.8 0) (unit 1)
+    (in_bom yes) (on_board yes)
+    (property "Reference" "#PWR0111" (id 0) (at 96.52 55.88 0)
+      (effects (font (size 1.27 1.27)) hide)
+    )
+    (property "Value" "GNDPWR" (id 1) (at 96.52 53.34 0)
+      (effects (font (size 0.381 0.381)))
+    )
+    (property "Footprint" "" (id 2) (at 96.52 52.07 0)
+      (effects (font (size 1.27 1.27)) hide)
+    )
+    (property "Datasheet" "" (id 3) (at 96.52 52.07 0)
       (effects (font (size 1.27 1.27)) hide)
     )
@@
       (reference "#PWR0104") (unit 1) (value "+5V") (footprint "")
     )
+    (path "/d9a142a0-10ac-44b2-9340-78628a0efc8f"
+      (reference "#PWR0105") (unit 1) (value "GNDPWR") (footprint "")
+    )
+    (path "/6dffb905-aeb2-45a0-8d0a-c9fece072daa"
+      (reference "#PWR0106") (unit 1) (value "GNDPWR") (footprint "")
+    )
+    (path "/42e2cea0-17f3-48f1-9378-5e2ba6972ab4"
+      (reference "#PWR0107") (unit 1) (value "GNDPWR") (footprint "")
+    )
+    (path "/7ba66d39-7263-4a63-9104-2d644caeb3a3"
+      (reference "#PWR0108") (unit 1) (value "GND") (footprint "")
+    )
     (path "/09e77cfc-c20b-4384-a667-11fef91a21dd"
       (reference "#PWR0109") (unit 1) (value "VBUS") (footprint "")
@@
       (reference "#PWR0110") (unit 1) (value "+5V") (footprint "")
     )
+    (path "/ff925d39-31af-4c1e-8be0-9f25e317ff13"
+      (reference "#PWR0111") (unit 1) (value "GNDPWR") (footprint "")
+    )
     (path "/0f5deb86-fcab-492d-905f-d8e47136ee96"
-      (reference "#PWR?") (unit 1) (value "GNDPWR") (footprint "")
-    )
-    (path "/42e2cea0-17f3-48f1-9378-5e2ba6972ab4"
-      (reference "#PWR?") (unit 1) (value "GNDPWR") (footprint "")
-    )
-    (path "/6dffb905-aeb2-45a0-8d0a-c9fece072daa"
-      (reference "#PWR?") (unit 1) (value "GNDPWR") (footprint "")
-    )
-    (path "/7ba66d39-7263-4a63-9104-2d644caeb3a3"
-      (reference "#PWR?") (unit 1) (value "GND") (footprint "")
+      (reference "#PWR0112") (unit 1) (value "GNDPWR") (footprint "")
+    )
+    (path "/dc0ac0fb-e92c-45ac-bb1a-94c4cf146b09"
+      (reference "#PWR0113") (unit 1) (value "GNDPWR") (footprint "")
     )
     (path "/a62db0bf-d79b-4255-b4f3-86b0890815cf"
-      (reference "#PWR?") (unit 1) (value "GNDPWR") (footprint "")
-    )
-    (path "/d9a142a0-10ac-44b2-9340-78628a0efc8f"
-      (reference "#PWR?") (unit 1) (value "GNDPWR") (footprint "")
-    )
-    (path "/dc0ac0fb-e92c-45ac-bb1a-94c4cf146b09"
-      (reference "#PWR?") (unit 1) (value "GNDPWR") (footprint "")
-    )
-    (path "/ff925d39-31af-4c1e-8be0-9f25e317ff13"
-      (reference "#PWR?") (unit 1) (value "GNDPWR") (footprint "")
+      (reference "#PWR0114") (unit 1) (value "GNDPWR") (footprint "")
     )
     (path "/062791e6-12f0-44fc-90f6-45f64ecdec87"
@@
     )
     (path "/22294464-5c73-43d3-ae56-8a26bed6f964"
-      (reference "H1") (unit 1) (value "MountingHole_Pad") (footprint "")
+      (reference "H1") (unit 1) (value "MountingHole_Pad") (footprint "MountingHole:MountingHole_2.2mm_M2_Pad")
     )
     (path "/ff6b3d40-632b-40fe-9881-f36d083abeb2"
-      (reference "H2") (unit 1) (value "MountingHole") (footprint "")
+      (reference "H2") (unit 1) (value "MountingHole") (footprint "MountingHole:MountingHole_2.2mm_M2_Pad")
     )
     (path "/d87e03a6-ee81-49b4-8c08-f15bda7dd13b"
-      (reference "H3") (unit 1) (value "MountingHole") (footprint "")
+      (reference "H3") (unit 1) (value "MountingHole") (footprint "MountingHole:MountingHole_2.2mm_M2_Pad")
     )
     (path "/18615ddf-d6ea-4001-aff0-38485a814a47"
-      (reference "H4") (unit 1) (value "MountingHole") (footprint "")
+      (reference "H4") (unit 1) (value "MountingHole") (footprint "MountingHole:MountingHole_2.2mm_M2_Pad")
     )
     (path "/f597188e-ece8-4dde-a990-5b3388b8413b"
