File: pcb/usbc_daughterboard/usbc64/usbc64.kicad_pcb (KiCad board)
At the start: 2 copper layers, 18 x 16.5 mm, 15 parts, among them J1 C-31-M12, J2 JST SH, U1 ESDALD05UG4

Commit message: connect MP pads to ground plane
Parts:
- R3: value 630 -> 630Ω
Changed lines of the file:
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@@
     (fp_line (start -1.5 -0.967893) (end -1 -1.675) (layer "F.Fab") (width 0.1))
     (fp_line (start -2 -1.675) (end -1.5 -0.967893) (layer "F.Fab") (width 0.1))
-    (pad "" smd roundrect (at 2.8 1.8) (size 1.2 1.8) (layers "F.Cu" "F.Paste" "F.Mask") (roundrect_rratio 0.208333))
-    (pad "" smd roundrect (at -2.8 1.8) (size 1.2 1.8) (layers "F.Cu" "F.Paste" "F.Mask") (roundrect_rratio 0.208333))
     (pad "1" smd roundrect (at -1.5 -2) (size 0.6 1.55) (layers "F.Cu" "F.Paste" "F.Mask") (roundrect_rratio 0.25)
       (net 7 "+5V") (pinfunction "Pin_1") (pintype "passive"))
@@
     (pad "4" smd roundrect (at 1.5 -2) (size 0.6 1.55) (layers "F.Cu" "F.Paste" "F.Mask") (roundrect_rratio 0.25)
       (net 1 "GND") (pinfunction "Pin_4") (pintype "passive"))
+    (pad "MP" smd roundrect (at 2.8 1.8) (size 1.2 1.8) (layers "F.Cu" "F.Paste" "F.Mask") (roundrect_rratio 0.208333)
+      (net 8 "GNDPWR") (pinfunction "MP") (pintype "power_in"))
+    (pad "MP" smd roundrect (at -2.8 1.8) (size 1.2 1.8) (layers "F.Cu" "F.Paste" "F.Mask") (roundrect_rratio 0.208333)
+      (net 8 "GNDPWR") (pinfunction "MP") (pintype "power_in"))
     (model "${REPO_3DMODEL_DIR}/SM04B-SRSS-TB.STEP"
       (offset (xyz 0 1.4 -0.3))
@@
       (effects (font (size 1 1) (thickness 0.15)))
     )
-    (fp_text value "630" (at 0 1.43) (layer "F.Fab")
-      (effects (font (size 1 1) (thickness 0.15)))
-    )
+    (fp_text value "630Ω" (at 0 1.43) (layer "F.Fab")
+      (effects (font (size 1 1) (thickness 0.15)))
+    )

Commit message: bidir zener diode value
Parts:
- D1: value D_TVS -> SMF8.5CA
Changed lines of the file:
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@@
       (effects (font (size 1 1) (thickness 0.2)))
     )
-    (fp_text value "D_TVS" (at 0 2.1 90) (layer "F.Fab")
+    (fp_text value "SMF8.5CA" (at 0 2.1 90) (layer "F.Fab")
       (effects (font (size 1 1) (thickness 0.15)))
     )
