File: pcb/usbc_daughterboard/usbc64/usbc64.kicad_pcb (KiCad board)
At the start: 2 copper layers, 18 x 16.5 mm, 15 parts, among them J1 C-31-M12, J2 JST SH, U1 ESDALD05UG4

Commit message: JLC order no. tag
Other:
- board text added: "JLCJLCJLCJLC"
Changed lines of the file:
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@@
     (property "Sheetname" "")
     (attr smd)
-    (fp_text reference "J1" (at 0 1.15) (layer "F.SilkS")
+    (fp_text reference "J1" (at 2.3 2.45) (layer "F.SilkS")
       (effects (font (size 1 1) (thickness 0.2)))
     )
@@
       (effects (font (size 1 1) (thickness 0.15)))
     )
-    (fp_line (start 4.7 2) (end 4.7 3.5) (layer "F.SilkS") (width 0.12))
     (fp_line (start -4.7 -1.9) (end -4.7 0.1) (layer "F.SilkS") (width 0.12))
-    (fp_line (start -4.7 2) (end -4.7 3.5) (layer "F.SilkS") (width 0.12))
     (fp_line (start 4.7 -1.9) (end 4.7 0.1) (layer "F.SilkS") (width 0.12))
     (fp_line (start -5 4) (end 5 4) (layer "F.CrtYd") (width 0.05))
@@
     (effects (font (size 1.5 1.5) (thickness 0.3)) (justify mirror))
   )
+  (gr_text "JLCJLCJLCJLC" (at 105 49.5 30) (layer "F.SilkS")
+    (effects (font (size 0.85 0.85) (thickness 0.2)))
+  )
   (segment (start 106.5 58.05) (end 106.85 58.4) (width 0.381) (layer "F.Cu") (net 1))

Commit message: remove jlcjlcjlcjlc
Other:
- board text removed: "JLCJLCJLCJLC"
Changed lines of the file:
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@@
     (property "Sheetname" "")
     (attr smd)
-    (fp_text reference "J1" (at 2.3 2.45) (layer "F.SilkS")
+    (fp_text reference "J1" (at 0 1.15) (layer "F.SilkS")
       (effects (font (size 1 1) (thickness 0.2)))
     )
@@
     (effects (font (size 1.5 1.5) (thickness 0.3)) (justify mirror))
   )
-  (gr_text "JLCJLCJLCJLC" (at 105 49.5 30) (layer "F.SilkS")
-    (effects (font (size 0.85 0.85) (thickness 0.2)))
-  )
   (segment (start 106.5 58.05) (end 106.85 58.4) (width 0.381) (layer "F.Cu") (net 1))

Commit message: usbc silk raster
Parts:
- added Ge: LOGO, BD:usbc_back_silkraster, B.Cu at (105.0, 54.7)
Other:
- board text removed: "beady"
- board text removed: "biddle"
