File: pcb/touchpad_daughterboard/cap64pcb.kicad_sch (KiCad schematic)
At the start: 30 parts, among them J1 SM04B_SURS_TF, Q1 BSS138, Q2 BSS138, U1 MPR121QR2, U2 SPX3819-3.3

Commit message: 0603 LED footprint
Parts:
- D1: footprint LED_SMD:LED_0805_2012Metric -> LED_SMD:LED_0603_1608Metric
Changed lines of the file:
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@@
+    (stroke (width 0) (type default) (color 0 0 0 0))
+  )
+  (wire (pts (xy 22.225 45.085) (xy 22.225 43.815))
+    (stroke (width 0) (type default) (color 0 0 0 0))
+  )
+  (wire (pts (xy 58.42 40.005) (xy 58.42 41.275))
+    (stroke (width 0) (type default) (color 0 0 0 0))
+  )
+  (wire (pts (xy 172.72 51.435) (xy 180.34 51.435))
+    (stroke (width 0) (type default) (color 0 0 0 0))
+  )
+  (wire (pts (xy 97.79 56.515) (xy 100.33 56.515))
+    (stroke (width 0) (type default) (color 0 0 0 0))
+  )
+  (wire (pts (xy 146.685 41.275) (xy 146.685 40.005))
+    (stroke (width 0) (type default) (color 0 0 0 0))
+  )
+  (wire (pts (xy 125.73 71.755) (xy 127 71.755))
+    (stroke (width 0) (type default) (color 0 0 0 0))
+  )
+  (wire (pts (xy 173.355 48.895) (xy 180.34 48.895))
+    (stroke (width 0) (type default) (color 0 0 0 0))
+  )
+  (wire (pts (xy 35.56 52.705) (xy 35.56 51.435))
+    (stroke (width 0) (type default) (color 0 0 0 0))
+  )
+  (wire (pts (xy 179.07 43.815) (xy 179.07 56.515))
     (stroke (width 0) (type default) (color 0 0 0 0))
   )
@@
     (stroke (width 0) (type default) (color 0 0 0 0))
   )
-  (wire (pts (xy 22.225 45.085) (xy 22.225 43.815))
-    (stroke (width 0) (type default) (color 0 0 0 0))
-  )
-  (wire (pts (xy 58.42 40.005) (xy 58.42 41.275))
-    (stroke (width 0) (type default) (color 0 0 0 0))
-  )
-  (wire (pts (xy 172.72 51.435) (xy 180.34 51.435))
-    (stroke (width 0) (type default) (color 0 0 0 0))
-  )
-  (wire (pts (xy 146.685 41.275) (xy 146.685 40.005))
-    (stroke (width 0) (type default) (color 0 0 0 0))
-  )
-  (wire (pts (xy 125.73 71.755) (xy 127 71.755))
-    (stroke (width 0) (type default) (color 0 0 0 0))
-  )
-  (wire (pts (xy 173.355 48.895) (xy 180.34 48.895))
-    (stroke (width 0) (type default) (color 0 0 0 0))
-  )
-  (wire (pts (xy 35.56 52.705) (xy 35.56 51.435))
-    (stroke (width 0) (type default) (color 0 0 0 0))
-  )
-  (wire (pts (xy 179.07 43.815) (xy 179.07 56.515))
-    (stroke (width 0) (type default) (color 0 0 0 0))
-  )
-  (wire (pts (xy 97.79 56.515) (xy 100.33 56.515))
+  (wire (pts (xy 90.805 46.355) (xy 90.805 56.515))
     (stroke (width 0) (type default) (color 0 0 0 0))
   )
@@
   )
   (wire (pts (xy 44.45 50.165) (xy 44.45 52.705))
-    (stroke (width 0) (type default) (color 0 0 0 0))
-  )
-  (wire (pts (xy 90.805 46.355) (xy 90.805 56.515))
     (stroke (width 0) (type default) (color 0 0 0 0))
   )
@@
       (effects (font (size 1.27 1.27)) (justify right))
     )
-    (property "Footprint" "LED_SMD:LED_0805_2012Metric" (id 2) (at 95.25 56.515 90)
+    (property "Footprint" "LED_SMD:LED_0603_1608Metric" (id 2) (at 95.25 56.515 90)
       (effects (font (size 1.27 1.27)) hide)
     )
@@
     )
     (path "/c99a01b3-5224-46b3-9237-a21f39c43bb5"
-      (reference "D1") (unit 1) (value "INT") (footprint "LED_SMD:LED_0805_2012Metric")
+      (reference "D1") (unit 1) (value "INT") (footprint "LED_SMD:LED_0603_1608Metric")
     )
     (path "/19d8f5e6-7917-4311-ae54-a6b4c084a96c"

Commit message: magnets with DRC errors lmao
Parts:
- added H1, H2: MountingHole, MountingHole:MountingHole_4mm, symbol Mechanical:MountingHole
Changed lines of the file:
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@@
     (pin "1")
+  )
+  (symbol (lib_id "Mechanical:MountingHole") (at 36.195 74.93 0) (unit 1)
+    (in_bom yes) (on_board yes) (fields_autoplaced)
+    (property "Reference" "H1" (id 0) (at 38.735 74.0953 0)
+      (effects (font (size 1.27 1.27)) (justify left))
+    )
+    (property "Value" "MountingHole" (id 1) (at 38.735 76.6322 0)
+      (effects (font (size 1.27 1.27)) (justify left))
+    )
+    (property "Footprint" "MountingHole:MountingHole_4mm" (id 2) (at 36.195 74.93 0)
+      (effects (font (size 1.27 1.27)) hide)
+    )
+    (property "Datasheet" "~" (id 3) (at 36.195 74.93 0)
+      (effects (font (size 1.27 1.27)) hide)
+    )
   )
   (symbol (lib_id "power:GND") (at 58.42 52.705 0) (unit 1)
@@
     (pin "1")
     (pin "2")
+  )
+  (symbol (lib_id "Mechanical:MountingHole") (at 36.195 80.645 0) (unit 1)
+    (in_bom yes) (on_board yes) (fields_autoplaced)
+    (property "Reference" "H2" (id 0) (at 38.735 79.8103 0)
+      (effects (font (size 1.27 1.27)) (justify left))
+    )
+    (property "Value" "MountingHole" (id 1) (at 38.735 82.3472 0)
+      (effects (font (size 1.27 1.27)) (justify left))
+    )
+    (property "Footprint" "MountingHole:MountingHole_4mm" (id 2) (at 36.195 80.645 0)
+      (effects (font (size 1.27 1.27)) hide)
+    )
+    (property "Datasheet" "~" (id 3) (at 36.195 80.645 0)
+      (effects (font (size 1.27 1.27)) hide)
+    )
   )
   (symbol (lib_id "power:+3V3") (at 161.925 40.005 0) (unit 1)
@@
       (reference "D1") (unit 1) (value "INT") (footprint "LED_SMD:LED_0603_1608Metric")
     )
+    (path "/293cdb1d-0389-4c2a-9ac9-1ee2cfc7ddb6"
+      (reference "H1") (unit 1) (value "MountingHole") (footprint "MountingHole:MountingHole_4mm")
+    )
+    (path "/6977b971-73fc-4aa6-af9f-63436b840f3d"
+      (reference "H2") (unit 1) (value "MountingHole") (footprint "MountingHole:MountingHole_4mm")
+    )
     (path "/19d8f5e6-7917-4311-ae54-a6b4c084a96c"

Commit message: MH values
Parts:
- H1, H2: value MountingHole -> MagnetHole
Changed lines of the file:
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@@
       (effects (font (size 1.27 1.27)) (justify left))
     )
-    (property "Value" "MountingHole" (id 1) (at 38.735 76.6322 0)
+    (property "Value" "MagnetHole" (id 1) (at 38.735 76.6322 0)
       (effects (font (size 1.27 1.27)) (justify left))
     )
@@
       (effects (font (size 1.27 1.27)) (justify left))
     )
-    (property "Value" "MountingHole" (id 1) (at 38.735 82.3472 0)
+    (property "Value" "MagnetHole" (id 1) (at 38.735 82.3472 0)
       (effects (font (size 1.27 1.27)) (justify left))
     )
@@
     )
     (path "/293cdb1d-0389-4c2a-9ac9-1ee2cfc7ddb6"
-      (reference "H1") (unit 1) (value "MountingHole") (footprint "MountingHole:MountingHole_4mm")
+      (reference "H1") (unit 1) (value "MagnetHole") (footprint "MountingHole:MountingHole_4mm")
     )
     (path "/6977b971-73fc-4aa6-af9f-63436b840f3d"
-      (reference "H2") (unit 1) (value "MountingHole") (footprint "MountingHole:MountingHole_4mm")
+      (reference "H2") (unit 1) (value "MagnetHole") (footprint "MountingHole:MountingHole_4mm")
     )
     (path "/19d8f5e6-7917-4311-ae54-a6b4c084a96c"

Commit message: 5pin jst sur
Parts:
- added M1: Motor_DC, symbol Motor:Motor_DC
- J1: footprint Connector_JST:JST_SUR_SM04B-SURS-TF_1x04-1MP_P0.80mm_Horizontal -> Connector_JST:JST_SUR_SM05B-SURS-TF_1x05-1MP_P0.80mm_Horizontal; symbol Connector_Generic:Conn_01x04 -> Connector_Generic:Conn_01x05
Connections:
- net GND: now also J1.3 (Pin_3), M1.2 (-); no longer J1.1 (Pin_1)
- net at Q1.3 (D): now also J1.4 (Pin_4); no longer J1.3 (Pin_3)
- net at Q2.3 (D): now also J1.5 (Pin_5); no longer J1.4 (Pin_4)
- new net VIB: J1.1 (Pin_1), M1.1 (+)
Changed lines of the file:
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@@
+    (stroke (width 0) (type default) (color 0 0 0 0))
+  )
+  (wire (pts (xy 173.99 78.105) (xy 173.99 79.375))
+    (stroke (width 0) (type default) (color 0 0 0 0))
+  )
+  (wire (pts (xy 158.75 78.105) (xy 160.02 78.105))
     (stroke (width 0) (type default) (color 0 0 0 0))
   )
@@
     (stroke (width 0) (type default) (color 0 0 0 0))
   )
+  (wire (pts (xy 177.8 46.355) (xy 177.8 56.515))
+    (stroke (width 0) (type default) (color 0 0 0 0))
+  )
   (wire (pts (xy 51.435 50.165) (xy 51.435 52.705))
     (stroke (width 0) (type default) (color 0 0 0 0))
@@
     (stroke (width 0) (type default) (color 0 0 0 0))
   )
-  (wire (pts (xy 175.895 40.005) (xy 175.895 46.355))
+  (wire (pts (xy 173.355 48.895) (xy 180.34 48.895))
     (stroke (width 0) (type default) (color 0 0 0 0))
   )
@@
     (stroke (width 0) (type default) (color 0 0 0 0))
   )
-  (wire (pts (xy 175.895 46.355) (xy 180.34 46.355))
-    (stroke (width 0) (type default) (color 0 0 0 0))
-  )
   (wire (pts (xy 44.45 43.815) (xy 44.45 45.085))
     (stroke (width 0) (type default) (color 0 0 0 0))
@@
     (stroke (width 0) (type default) (color 0 0 0 0))
   )
-  (wire (pts (xy 172.72 51.435) (xy 180.34 51.435))
-    (stroke (width 0) (type default) (color 0 0 0 0))
-  )
   (wire (pts (xy 97.79 56.515) (xy 100.33 56.515))
     (stroke (width 0) (type default) (color 0 0 0 0))
@@
     (stroke (width 0) (type default) (color 0 0 0 0))
   )
-  (wire (pts (xy 173.355 48.895) (xy 180.34 48.895))
+  (wire (pts (xy 173.355 40.005) (xy 173.355 43.815))
     (stroke (width 0) (type default) (color 0 0 0 0))
   )
@@
     (stroke (width 0) (type default) (color 0 0 0 0))
   )
-  (wire (pts (xy 179.07 43.815) (xy 179.07 56.515))
-    (stroke (width 0) (type default) (color 0 0 0 0))
-  )
   (wire (pts (xy 90.805 56.515) (xy 92.71 56.515))
     (stroke (width 0) (type default) (color 0 0 0 0))
@@
     (stroke (width 0) (type default) (color 0 0 0 0))
   )
-  (wire (pts (xy 158.115 54.61) (xy 172.72 54.61))
+  (wire (pts (xy 158.115 54.61) (xy 173.355 54.61))
     (stroke (width 0) (type default) (color 0 0 0 0))
   )
@@
     (stroke (width 0) (type default) (color 0 0 0 0))
   )
+  (wire (pts (xy 172.72 78.105) (xy 173.99 78.105))
+    (stroke (width 0) (type default) (color 0 0 0 0))
+  )
   (wire (pts (xy 22.225 50.165) (xy 22.225 52.705))
     (stroke (width 0) (type default) (color 0 0 0 0))
@@
     (stroke (width 0) (type default) (color 0 0 0 0))
   )
-  (wire (pts (xy 180.34 43.815) (xy 179.07 43.815))
-    (stroke (width 0) (type default) (color 0 0 0 0))
-  )
   (wire (pts (xy 146.685 54.61) (xy 147.955 54.61))
     (stroke (width 0) (type default) (color 0 0 0 0))
   )
+  (wire (pts (xy 177.8 46.355) (xy 180.34 46.355))
+    (stroke (width 0) (type default) (color 0 0 0 0))
+  )
   (wire (pts (xy 113.03 40.005) (xy 113.03 41.275))
     (stroke (width 0) (type default) (color 0 0 0 0))
@@
     (stroke (width 0) (type default) (color 0 0 0 0))
   )
+  (wire (pts (xy 173.355 43.815) (xy 180.34 43.815))
+    (stroke (width 0) (type default) (color 0 0 0 0))
+  )
   (wire (pts (xy 161.925 48.895) (xy 163.195 48.895))
     (stroke (width 0) (type default) (color 0 0 0 0))
@@
     (stroke (width 0) (type default) (color 0 0 0 0))
   )
-  (wire (pts (xy 172.72 54.61) (xy 172.72 51.435))
+  (wire (pts (xy 173.355 54.61) (xy 173.355 51.435))
     (stroke (width 0) (type default) (color 0 0 0 0))
   )
@@
     (stroke (width 0) (type default) (color 0 0 0 0))
   )
+  (wire (pts (xy 158.75 76.835) (xy 158.75 78.105))
+    (stroke (width 0) (type default) (color 0 0 0 0))
+  )
   (wire (pts (xy 168.275 40.005) (xy 168.275 41.275))
     (stroke (width 0) (type default) (color 0 0 0 0))
   )
   (wire (pts (xy 125.73 56.515) (xy 127 56.515))
+    (stroke (width 0) (type default) (color 0 0 0 0))
+  )
+  (wire (pts (xy 173.355 51.435) (xy 180.34 51.435))
     (stroke (width 0) (type default) (color 0 0 0 0))
   )
@@
     )
   )
+  (global_label "VIB" (shape input) (at 158.75 76.835 90) (fields_autoplaced)
+    (effects (font (size 1.27 1.27)) (justify left))
+    (property "Intersheet References" "${INTERSHEET_REFS}" (id 0) (at 158.6706 71.4586 90)
+      (effects (font (size 1.27 1.27)) (justify left) hide)
+    )
+  )
   (global_label "SCL" (shape input) (at 145.415 54.61 180) (fields_autoplaced)
     (effects (font (size 1.27 1.27)) (justify right))
@@
     )
   )
+  (global_label "VIB" (shape input) (at 180.34 41.275 180) (fields_autoplaced)
+    (effects (font (size 1.27 1.27)) (justify right))
+    (property "Intersheet References" "${INTERSHEET_REFS}" (id 0) (at 174.9636 41.3544 0)
+      (effects (font (size 1.27 1.27)) (justify right) hide)
+    )
+  )
   (global_label "SDA" (shape input) (at 81.28 56.515 180) (fields_autoplaced)
     (effects (font (size 1.27 1.27)) (justify right))
@@
     (pin "1")
   )
-  (symbol (lib_id "Connector_Generic:Conn_01x04") (at 185.42 46.355 0) (unit 1)
+  (symbol (lib_id "Connector_Generic:Conn_01x05") (at 185.42 46.355 0) (unit 1)
     (in_bom yes) (on_board yes)
     (property "Reference" "J1" (id 0) (at 184.15 41.275 0)
@@
       (effects (font (size 1.27 1.27)) (justify left))
     )
-    (property "Footprint" "Connector_JST:JST_SUR_SM04B-SURS-TF_1x04-1MP_P0.80mm_Horizontal" (id 2) (at 185.42 46.355 0)
+    (property "Footprint" "Connector_JST:JST_SUR_SM05B-SURS-TF_1x05-1MP_P0.80mm_Horizontal" (id 2) (at 185.42 46.355 0)
       (effects (font (size 1.27 1.27)) hide)
     )
@@
     (pin "3")
     (pin "4")
+    (pin "5")
     (pin "MP")
   )
@@
     (pin "1")
   )
-  (symbol (lib_id "power:GND") (at 179.07 56.515 0) (unit 1)
-    (in_bom yes) (on_board yes)
-    (property "Reference" "#PWR0114" (id 0) (at 179.07 62.865 0)
-      (effects (font (size 1.27 1.27)) hide)
-    )
-    (property "Value" "GND" (id 1) (at 179.07 60.325 0))
-    (property "Footprint" "" (id 2) (at 179.07 56.515 0)
-      (effects (font (size 1.27 1.27)) hide)
-    )
-    (property "Datasheet" "" (id 3) (at 179.07 56.515 0)
+  (symbol (lib_id "power:GND") (at 177.8 56.515 0) (unit 1)
+    (in_bom yes) (on_board yes)
+    (property "Reference" "#PWR0114" (id 0) (at 177.8 62.865 0)
+      (effects (font (size 1.27 1.27)) hide)
+    )
+    (property "Value" "GND" (id 1) (at 177.8 60.325 0))
+    (property "Footprint" "" (id 2) (at 177.8 56.515 0)
+      (effects (font (size 1.27 1.27)) hide)
+    )
+    (property "Datasheet" "" (id 3) (at 177.8 56.515 0)
       (effects (font (size 1.27 1.27)) hide)
     )
@@
     (pin "2")
     (pin "3")
+  )
+  (symbol (lib_id "power:GND") (at 173.99 79.375 0) (unit 1)
+    (in_bom yes) (on_board yes)
+    (property "Reference" "#PWR0122" (id 0) (at 173.99 85.725 0)
+      (effects (font (size 1.27 1.27)) hide)
+    )
+    (property "Value" "GND" (id 1) (at 173.99 83.185 0))
+    (property "Footprint" "" (id 2) (at 173.99 79.375 0)
+      (effects (font (size 1.27 1.27)) hide)
+    )
+    (property "Datasheet" "" (id 3) (at 173.99 79.375 0)
+      (effects (font (size 1.27 1.27)) hide)
+    )
+    (pin "1")
   )
   (symbol (lib_id "power:+3V3") (at 82.55 40.005 0) (unit 1)
@@
     (pin "1")
   )
-  (symbol (lib_id "power:VCC") (at 175.895 40.005 0) (unit 1)
-    (in_bom yes) (on_board yes)
-    (property "Reference" "#PWR0117" (id 0) (at 175.895 43.815 0)
-      (effects (font (size 1.27 1.27)) hide)
-    )
-    (property "Value" "VCC" (id 1) (at 175.895 36.195 0))
-    (property "Footprint" "" (id 2) (at 175.895 40.005 0)
-      (effects (font (size 1.27 1.27)) hide)
-    )
-    (property "Datasheet" "" (id 3) (at 175.895 40.005 0)
+  (symbol (lib_id "Motor:Motor_DC") (at 165.1 78.105 90) (unit 1)
+    (in_bom yes) (on_board yes) (fields_autoplaced)
+    (property "Reference" "M1" (id 0) (at 167.64 71.154 90))
+    (property "Value" "Motor_DC" (id 1) (at 167.64 73.6909 90))
+    (property "Footprint" "" (id 2) (at 167.386 78.105 0)
+      (effects (font (size 1.27 1.27)) hide)
+    )
+    (property "Datasheet" "~" (id 3) (at 167.386 78.105 0)
+      (effects (font (size 1.27 1.27)) hide)
+    )
+    (pin "1")
+    (pin "2")
+  )
+  (symbol (lib_id "power:VCC") (at 173.355 40.005 0) (unit 1)
+    (in_bom yes) (on_board yes)
+    (property "Reference" "#PWR0117" (id 0) (at 173.355 43.815 0)
+      (effects (font (size 1.27 1.27)) hide)
+    )
+    (property "Value" "VCC" (id 1) (at 173.355 36.195 0))
+    (property "Footprint" "" (id 2) (at 173.355 40.005 0)
+      (effects (font (size 1.27 1.27)) hide)
+    )
+    (property "Datasheet" "" (id 3) (at 173.355 40.005 0)
       (effects (font (size 1.27 1.27)) hide)
     )
@@
       (reference "#PWR0121") (unit 1) (value "GND") (footprint "")
     )
+    (path "/987019a0-e790-4917-98b6-99b6a2c96f3d"
+      (reference "#PWR0122") (unit 1) (value "GND") (footprint "")
+    )
     (path "/f135c53c-386c-4051-aa9a-f8f2f6913b14"
       (reference "C1") (unit 1) (value "10uF") (footprint "Capacitor_SMD:C_0805_2012Metric")
@@
     )
     (path "/19d8f5e6-7917-4311-ae54-a6b4c084a96c"
-      (reference "J1") (unit 1) (value "SM04B_SURS_TF") (footprint "Connector_JST:JST_SUR_SM04B-SURS-TF_1x04-1MP_P0.80mm_Horizontal")
+      (reference "J1") (unit 1) (value "SM04B_SURS_TF") (footprint "Connector_JST:JST_SUR_SM05B-SURS-TF_1x05-1MP_P0.80mm_Horizontal")
     )
     (path "/fbb40797-6e54-4738-a17f-8e91819242d1"
       (reference "JP1") (unit 1) (value "SolderJumper_3_Open") (footprint "Jumper:SolderJumper-3_P1.3mm_Open_RoundedPad1.0x1.5mm_NumberLabels")
     )
+    (path "/ce6cb472-2467-4bd4-944e-2d52e18bda4b"
+      (reference "M1") (unit 1) (value "Motor_DC") (footprint "")
+    )
     (path "/4df03174-9603-43d2-88cc-bd6346b3f204"

Commit message: reorder and reroute connector
Connections:
- net GND: now also J1.2 (Pin_2); no longer J1.3 (Pin_3)
- net VCC: now also J1.1 (Pin_1); no longer J1.2 (Pin_2)
- net VIB: now also J1.3 (Pin_3); no longer J1.1 (Pin_1)
Changed lines of the file:
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@@
-    (stroke (width 0) (type default) (color 0 0 0 0))
-  )
-  (wire (pts (xy 177.8 46.355) (xy 177.8 56.515))
     (stroke (width 0) (type default) (color 0 0 0 0))
   )
@@
     (stroke (width 0) (type default) (color 0 0 0 0))
   )
+  (wire (pts (xy 177.8 40.005) (xy 177.8 41.275))
+    (stroke (width 0) (type default) (color 0 0 0 0))
+  )
   (wire (pts (xy 82.55 66.675) (xy 82.55 83.185))
     (stroke (width 0) (type default) (color 0 0 0 0))
@@
     (stroke (width 0) (type default) (color 0 0 0 0))
   )
-  (wire (pts (xy 173.355 40.005) (xy 173.355 43.815))
-    (stroke (width 0) (type default) (color 0 0 0 0))
-  )
   (wire (pts (xy 35.56 52.705) (xy 35.56 51.435))
     (stroke (width 0) (type default) (color 0 0 0 0))
@@
     (stroke (width 0) (type default) (color 0 0 0 0))
   )
+  (wire (pts (xy 177.8 41.275) (xy 180.34 41.275))
+    (stroke (width 0) (type default) (color 0 0 0 0))
+  )
   (wire (pts (xy 51.435 41.275) (xy 58.42 41.275))
     (stroke (width 0) (type default) (color 0 0 0 0))
@@
     (stroke (width 0) (type default) (color 0 0 0 0))
   )
+  (wire (pts (xy 180.34 43.815) (xy 177.8 43.815))
+    (stroke (width 0) (type default) (color 0 0 0 0))
+  )
   (wire (pts (xy 185.42 55.245) (xy 185.42 56.515))
     (stroke (width 0) (type default) (color 0 0 0 0))
@@
     (stroke (width 0) (type default) (color 0 0 0 0))
   )
-  (wire (pts (xy 177.8 46.355) (xy 180.34 46.355))
-    (stroke (width 0) (type default) (color 0 0 0 0))
-  )
   (wire (pts (xy 113.03 40.005) (xy 113.03 41.275))
     (stroke (width 0) (type default) (color 0 0 0 0))
@@
     (stroke (width 0) (type default) (color 0 0 0 0))
   )
-  (wire (pts (xy 173.355 43.815) (xy 180.34 43.815))
-    (stroke (width 0) (type default) (color 0 0 0 0))
-  )
   (wire (pts (xy 161.925 48.895) (xy 163.195 48.895))
     (stroke (width 0) (type default) (color 0 0 0 0))
@@
     (stroke (width 0) (type default) (color 0 0 0 0))
   )
+  (wire (pts (xy 173.355 46.355) (xy 180.34 46.355))
+    (stroke (width 0) (type default) (color 0 0 0 0))
+  )
   (wire (pts (xy 125.73 59.055) (xy 127 59.055))
     (stroke (width 0) (type default) (color 0 0 0 0))
@@
     (stroke (width 0) (type default) (color 0 0 0 0))
   )
+  (wire (pts (xy 173.355 44.45) (xy 173.355 46.355))
+    (stroke (width 0) (type default) (color 0 0 0 0))
+  )
   (wire (pts (xy 173.355 51.435) (xy 180.34 51.435))
+    (stroke (width 0) (type default) (color 0 0 0 0))
+  )
+  (wire (pts (xy 177.8 43.815) (xy 177.8 56.515))
     (stroke (width 0) (type default) (color 0 0 0 0))
   )
@@
     )
   )
-  (global_label "VIB" (shape input) (at 180.34 41.275 180) (fields_autoplaced)
-    (effects (font (size 1.27 1.27)) (justify right))
-    (property "Intersheet References" "${INTERSHEET_REFS}" (id 0) (at 174.9636 41.3544 0)
-      (effects (font (size 1.27 1.27)) (justify right) hide)
+  (global_label "VIB" (shape input) (at 173.355 44.45 90) (fields_autoplaced)
+    (effects (font (size 1.27 1.27)) (justify left))
+    (property "Intersheet References" "${INTERSHEET_REFS}" (id 0) (at 173.2756 39.0736 90)
+      (effects (font (size 1.27 1.27)) (justify left) hide)
     )
   )
@@
     (pin "1")
   )
-  (symbol (lib_id "power:GND") (at 177.8 56.515 0) (unit 1)
+  (symbol (lib_id "power:GND") (at 177.8 56.515 0) (mirror y) (unit 1)
     (in_bom yes) (on_board yes)
     (property "Reference" "#PWR0114" (id 0) (at 177.8 62.865 0)
@@
     (pin "2")
   )
-  (symbol (lib_id "power:VCC") (at 173.355 40.005 0) (unit 1)
-    (in_bom yes) (on_board yes)
-    (property "Reference" "#PWR0117" (id 0) (at 173.355 43.815 0)
-      (effects (font (size 1.27 1.27)) hide)
-    )
-    (property "Value" "VCC" (id 1) (at 173.355 36.195 0))
-    (property "Footprint" "" (id 2) (at 173.355 40.005 0)
-      (effects (font (size 1.27 1.27)) hide)
-    )
-    (property "Datasheet" "" (id 3) (at 173.355 40.005 0)
-      (effects (font (size 1.27 1.27)) hide)
-    )
+  (symbol (lib_id "power:VCC") (at 177.8 40.005 0) (unit 1)
+    (in_bom yes) (on_board yes)
+    (property "Reference" "#PWR0117" (id 0) (at 177.8 43.815 0)
+      (effects (font (size 1.27 1.27)) hide)
+    )
+    (property "Value" "VCC" (id 1) (at 177.8 36.195 0))
+    (property "Footprint" "" (id 2) (at 177.8 40.005 0)
+      (effects (font (size 1.27 1.27)) hide)
+    )
+    (property "Datasheet" "" (id 3) (at 177.8 40.005 0)
+      (effects (font (size 1.27 1.27)) hide)
+    )

Commit message: space made for coin motor
Parts:
- TP13, TP14: footprint TestPoint:TestPoint_Pad_2.0x2.0mm -> TestPoint:TestPoint_Pad_D1.0mm
Changed lines of the file:
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@@
       (effects (font (size 1.27 1.27)) (justify left) hide)
     )
-    (property "Footprint" "TestPoint:TestPoint_Pad_2.0x2.0mm" (id 2) (at 72.39 45.085 0)
+    (property "Footprint" "TestPoint:TestPoint_Pad_D1.0mm" (id 2) (at 72.39 45.085 0)
       (effects (font (size 1.27 1.27)) hide)
     )
@@
       (effects (font (size 1.27 1.27)) (justify right) hide)
     )
-    (property "Footprint" "TestPoint:TestPoint_Pad_2.0x2.0mm" (id 2) (at 77.47 45.085 0)
+    (property "Footprint" "TestPoint:TestPoint_Pad_D1.0mm" (id 2) (at 77.47 45.085 0)
       (effects (font (size 1.27 1.27)) hide)
     )
@@
     )
     (path "/fd00f671-a567-4561-b2a9-081b479a0835"
-      (reference "TP13") (unit 1) (value "b") (footprint "TestPoint:TestPoint_Pad_2.0x2.0mm")
+      (reference "TP13") (unit 1) (value "b") (footprint "TestPoint:TestPoint_Pad_D1.0mm")
     )
     (path "/681b5193-51cf-4708-8ba4-9c277717a057"
-      (reference "TP14") (unit 1) (value "d") (footprint "TestPoint:TestPoint_Pad_2.0x2.0mm")
+      (reference "TP14") (unit 1) (value "d") (footprint "TestPoint:TestPoint_Pad_D1.0mm")
     )
     (path "/c8c3ab22-4b33-4bf7-93a7-fa49e1af3364"
