File: pcb/touchpad_daughterboard/cap64pcb.kicad_sch (KiCad schematic)
At the start: 33 parts, among them J1 SM04B_SURS_TF, M1 Motor_DC, Q1 BSS138, Q2 BSS138, U1 MPR121QR2, U2 SPX3819-3.3

Commit message: ERM symbol/footprint/3d model
Parts:
- removed M1: Motor_DC, symbol Motor:Motor_DC
- added M1: Coin_Motor, coinERM:VC1018B001L, symbol coinERM:Coin_Motor
- added TP15: +, TestPoint:TestPoint_Pad_D1.0mm, symbol Connector:TestPoint
- added TP16: -, TestPoint:TestPoint_Pad_D1.0mm, symbol Connector:TestPoint
Connections:
- net GND: now also TP16.1
- net VIB: now also TP15.1
Other:
- moved on the sheet: H1, H2
Changed lines of the file:
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@@
+    (stroke (width 0) (type default) (color 0 0 0 0))
+  )
+  (wire (pts (xy 153.67 71.755) (xy 154.94 71.755))
     (stroke (width 0) (type default) (color 0 0 0 0))
   )
@@
     (stroke (width 0) (type default) (color 0 0 0 0))
   )
-  (wire (pts (xy 173.99 78.105) (xy 173.99 79.375))
-    (stroke (width 0) (type default) (color 0 0 0 0))
-  )
-  (wire (pts (xy 158.75 78.105) (xy 160.02 78.105))
-    (stroke (width 0) (type default) (color 0 0 0 0))
-  )
   (wire (pts (xy 125.73 74.295) (xy 127 74.295))
     (stroke (width 0) (type default) (color 0 0 0 0))
@@
     (stroke (width 0) (type default) (color 0 0 0 0))
   )
+  (wire (pts (xy 153.67 75.565) (xy 154.94 75.565))
+    (stroke (width 0) (type default) (color 0 0 0 0))
+  )
   (wire (pts (xy 97.79 56.515) (xy 100.33 56.515))
     (stroke (width 0) (type default) (color 0 0 0 0))
@@
     (stroke (width 0) (type default) (color 0 0 0 0))
   )
-  (wire (pts (xy 172.72 78.105) (xy 173.99 78.105))
-    (stroke (width 0) (type default) (color 0 0 0 0))
-  )
   (wire (pts (xy 22.225 50.165) (xy 22.225 52.705))
     (stroke (width 0) (type default) (color 0 0 0 0))
@@
     (stroke (width 0) (type default) (color 0 0 0 0))
   )
+  (wire (pts (xy 153.67 76.835) (xy 153.67 75.565))
+    (stroke (width 0) (type default) (color 0 0 0 0))
+  )
   (wire (pts (xy 161.925 40.005) (xy 161.925 41.275))
     (stroke (width 0) (type default) (color 0 0 0 0))
@@
   )
   (wire (pts (xy 22.225 43.815) (xy 27.94 43.815))
-    (stroke (width 0) (type default) (color 0 0 0 0))
-  )
-  (wire (pts (xy 158.75 76.835) (xy 158.75 78.105))
     (stroke (width 0) (type default) (color 0 0 0 0))
   )
@@
     )
   )
-  (global_label "VIB" (shape input) (at 158.75 76.835 90) (fields_autoplaced)
-    (effects (font (size 1.27 1.27)) (justify left))
-    (property "Intersheet References" "${INTERSHEET_REFS}" (id 0) (at 158.6706 71.4586 90)
-      (effects (font (size 1.27 1.27)) (justify left) hide)
+  (global_label "VIB" (shape input) (at 153.67 71.755 180) (fields_autoplaced)
+    (effects (font (size 1.27 1.27)) (justify right))
+    (property "Intersheet References" "${INTERSHEET_REFS}" (id 0) (at 148.2936 71.8344 0)
+      (effects (font (size 1.27 1.27)) (justify right) hide)
     )
   )
@@
     (pin "MP")
   )
+  (symbol (lib_id "coinERM:Coin_Motor") (at 167.005 73.66 0) (unit 1)
+    (in_bom yes) (on_board yes)
+    (property "Reference" "M1" (id 0) (at 165.735 73.66 0)
+      (effects (font (size 1.27 1.27)) (justify left))
+    )
+    (property "Value" "Coin_Motor" (id 1) (at 172.085 73.66 0)
+      (effects (font (size 1.27 1.27)) (justify left))
+    )
+    (property "Footprint" "coinERM:VC1018B001L" (id 2) (at 167.005 73.66 0)
+      (effects (font (size 1.27 1.27)) hide)
+    )
+    (property "Datasheet" "" (id 3) (at 167.005 73.66 0)
+      (effects (font (size 1.27 1.27)) hide)
+    )
+  )
   (symbol (lib_id "Regulator_Linear:SPX3819M5-L-3-3") (at 35.56 43.815 0) (unit 1)
     (in_bom yes) (on_board yes)
@@
     (pin "1")
   )
-  (symbol (lib_id "Mechanical:MountingHole") (at 36.195 74.93 0) (unit 1)
+  (symbol (lib_id "Mechanical:MountingHole") (at 38.735 71.12 0) (unit 1)
     (in_bom yes) (on_board yes) (fields_autoplaced)
-    (property "Reference" "H1" (id 0) (at 38.735 74.0953 0)
-      (effects (font (size 1.27 1.27)) (justify left))
-    )
-    (property "Value" "MagnetHole" (id 1) (at 38.735 76.6322 0)
-      (effects (font (size 1.27 1.27)) (justify left))
-    )
-    (property "Footprint" "MountingHole:MountingHole_4mm" (id 2) (at 36.195 74.93 0)
-      (effects (font (size 1.27 1.27)) hide)
-    )
-    (property "Datasheet" "~" (id 3) (at 36.195 74.93 0)
+    (property "Reference" "H1" (id 0) (at 41.275 70.2853 0)
+      (effects (font (size 1.27 1.27)) (justify left))
+    )
+    (property "Value" "MagnetHole" (id 1) (at 41.275 72.8222 0)
+      (effects (font (size 1.27 1.27)) (justify left))
+    )
+    (property "Footprint" "MountingHole:MountingHole_4mm" (id 2) (at 38.735 71.12 0)
+      (effects (font (size 1.27 1.27)) hide)
+    )
+    (property "Datasheet" "~" (id 3) (at 38.735 71.12 0)
       (effects (font (size 1.27 1.27)) hide)
     )
@@
     (pin "2")
   )
-  (symbol (lib_id "Mechanical:MountingHole") (at 36.195 80.645 0) (unit 1)
+  (symbol (lib_id "Mechanical:MountingHole") (at 38.735 76.835 0) (unit 1)
     (in_bom yes) (on_board yes) (fields_autoplaced)
-    (property "Reference" "H2" (id 0) (at 38.735 79.8103 0)
-      (effects (font (size 1.27 1.27)) (justify left))
-    )
-    (property "Value" "MagnetHole" (id 1) (at 38.735 82.3472 0)
-      (effects (font (size 1.27 1.27)) (justify left))
-    )
-    (property "Footprint" "MountingHole:MountingHole_4mm" (id 2) (at 36.195 80.645 0)
-      (effects (font (size 1.27 1.27)) hide)
-    )
-    (property "Datasheet" "~" (id 3) (at 36.195 80.645 0)
+    (property "Reference" "H2" (id 0) (at 41.275 76.0003 0)
+      (effects (font (size 1.27 1.27)) (justify left))
+    )
+    (property "Value" "MagnetHole" (id 1) (at 41.275 78.5372 0)
+      (effects (font (size 1.27 1.27)) (justify left))
+    )
+    (property "Footprint" "MountingHole:MountingHole_4mm" (id 2) (at 38.735 76.835 0)
+      (effects (font (size 1.27 1.27)) hide)
+    )
+    (property "Datasheet" "~" (id 3) (at 38.735 76.835 0)
       (effects (font (size 1.27 1.27)) hide)
     )
@@
     (pin "3")
   )
-  (symbol (lib_id "power:GND") (at 173.99 79.375 0) (unit 1)
-    (in_bom yes) (on_board yes)
-    (property "Reference" "#PWR0122" (id 0) (at 173.99 85.725 0)
-      (effects (font (size 1.27 1.27)) hide)
-    )
-    (property "Value" "GND" (id 1) (at 173.99 83.185 0))
-    (property "Footprint" "" (id 2) (at 173.99 79.375 0)
-      (effects (font (size 1.27 1.27)) hide)
-    )
-    (property "Datasheet" "" (id 3) (at 173.99 79.375 0)
+  (symbol (lib_id "Connector:TestPoint") (at 154.94 75.565 270) (unit 1)
+    (in_bom yes) (on_board yes)
+    (property "Reference" "TP16" (id 0) (at 156.21 77.47 90)
+      (effects (font (size 1.27 1.27)) (justify left))
+    )
+    (property "Value" "-" (id 1) (at 159.639 77.2672 90)
+      (effects (font (size 1.27 1.27)) (justify left) hide)
+    )
+    (property "Footprint" "TestPoint:TestPoint_Pad_D1.0mm" (id 2) (at 154.94 80.645 0)
+      (effects (font (size 1.27 1.27)) hide)
+    )
+    (property "Datasheet" "~" (id 3) (at 154.94 80.645 0)
+      (effects (font (size 1.27 1.27)) hide)
+    )
+    (pin "1")
+  )
+  (symbol (lib_id "power:GND") (at 153.67 76.835 0) (unit 1)
+    (in_bom yes) (on_board yes)
+    (property "Reference" "#PWR0122" (id 0) (at 153.67 83.185 0)
+      (effects (font (size 1.27 1.27)) hide)
+    )
+    (property "Value" "GND" (id 1) (at 153.67 80.645 0))
+    (property "Footprint" "" (id 2) (at 153.67 76.835 0)
+      (effects (font (size 1.27 1.27)) hide)
+    )
+    (property "Datasheet" "" (id 3) (at 153.67 76.835 0)
       (effects (font (size 1.27 1.27)) hide)
     )
@@
     (pin "1")
   )
-  (symbol (lib_id "Motor:Motor_DC") (at 165.1 78.105 90) (unit 1)
-    (in_bom yes) (on_board yes) (fields_autoplaced)
-    (property "Reference" "M1" (id 0) (at 167.64 71.154 90))
-    (property "Value" "Motor_DC" (id 1) (at 167.64 73.6909 90))
-    (property "Footprint" "" (id 2) (at 167.386 78.105 0)
-      (effects (font (size 1.27 1.27)) hide)
-    )
-    (property "Datasheet" "~" (id 3) (at 167.386 78.105 0)
-      (effects (font (size 1.27 1.27)) hide)
-    )
-    (pin "1")
-    (pin "2")
-  )
   (symbol (lib_id "power:VCC") (at 177.8 40.005 0) (unit 1)
     (in_bom yes) (on_board yes)
@@
     )
     (property "Datasheet" "" (id 3) (at 177.8 40.005 0)
+      (effects (font (size 1.27 1.27)) hide)
+    )
+    (pin "1")
+  )
+  (symbol (lib_id "Connector:TestPoint") (at 154.94 71.755 270) (unit 1)
+    (in_bom yes) (on_board yes)
+    (property "Reference" "TP15" (id 0) (at 156.21 69.85 90)
+      (effects (font (size 1.27 1.27)) (justify left))
+    )
+    (property "Value" "+" (id 1) (at 159.639 73.4572 90)
+      (effects (font (size 1.27 1.27)) (justify left) hide)
+    )
+    (property "Footprint" "TestPoint:TestPoint_Pad_D1.0mm" (id 2) (at 154.94 76.835 0)
+      (effects (font (size 1.27 1.27)) hide)
+    )
+    (property "Datasheet" "~" (id 3) (at 154.94 76.835 0)
       (effects (font (size 1.27 1.27)) hide)
     )
@@
       (reference "JP1") (unit 1) (value "SolderJumper_3_Open") (footprint "Jumper:SolderJumper-3_P1.3mm_Open_RoundedPad1.0x1.5mm_NumberLabels")
     )
-    (path "/ce6cb472-2467-4bd4-944e-2d52e18bda4b"
-      (reference "M1") (unit 1) (value "Motor_DC") (footprint "")
+    (path "/1a7cbff0-a3bd-43cd-a4f2-8cb479e17f7b"
+      (reference "M1") (unit 1) (value "Coin_Motor") (footprint "coinERM:VC1018B001L")
     )
     (path "/4df03174-9603-43d2-88cc-bd6346b3f204"
@@
       (reference "TP14") (unit 1) (value "d") (footprint "TestPoint:TestPoint_Pad_D1.0mm")
     )
+    (path "/eaca30a7-2643-4e7e-a256-0b34720af638"
+      (reference "TP15") (unit 1) (value "+") (footprint "TestPoint:TestPoint_Pad_D1.0mm")
+    )
+    (path "/94ba82fd-b8f6-446f-bba5-bba684667285"
+      (reference "TP16") (unit 1) (value "-") (footprint "TestPoint:TestPoint_Pad_D1.0mm")
+    )
     (path "/c8c3ab22-4b33-4bf7-93a7-fa49e1af3364"

Commit message: erm footprint update, all routed, no errors
Parts:
- TP15, TP16: footprint TestPoint:TestPoint_Pad_D1.0mm -> TestPoint:TestPoint_Pad_1.0x1.0mm
Changed lines of the file:
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@@
       (effects (font (size 1.27 1.27)) (justify left) hide)
     )
-    (property "Footprint" "TestPoint:TestPoint_Pad_D1.0mm" (id 2) (at 154.94 80.645 0)
+    (property "Footprint" "TestPoint:TestPoint_Pad_1.0x1.0mm" (id 2) (at 154.94 80.645 0)
       (effects (font (size 1.27 1.27)) hide)
     )
@@
       (effects (font (size 1.27 1.27)) (justify left) hide)
     )
-    (property "Footprint" "TestPoint:TestPoint_Pad_D1.0mm" (id 2) (at 154.94 76.835 0)
+    (property "Footprint" "TestPoint:TestPoint_Pad_1.0x1.0mm" (id 2) (at 154.94 76.835 0)
       (effects (font (size 1.27 1.27)) hide)
     )
@@
     )
     (path "/eaca30a7-2643-4e7e-a256-0b34720af638"
-      (reference "TP15") (unit 1) (value "+") (footprint "TestPoint:TestPoint_Pad_D1.0mm")
+      (reference "TP15") (unit 1) (value "+") (footprint "TestPoint:TestPoint_Pad_1.0x1.0mm")
     )
     (path "/94ba82fd-b8f6-446f-bba5-bba684667285"
-      (reference "TP16") (unit 1) (value "-") (footprint "TestPoint:TestPoint_Pad_D1.0mm")
+      (reference "TP16") (unit 1) (value "-") (footprint "TestPoint:TestPoint_Pad_1.0x1.0mm")
     )
     (path "/c8c3ab22-4b33-4bf7-93a7-fa49e1af3364"
