File: pcb/touchpad_daughterboard/cap64pcb.kicad_sch (KiCad schematic)
At the start: 35 parts, among them J1 SM04B_SURS_TF, M1 Coin_Motor, Q1 BSS138, Q2 BSS138, U1 MPR121QR2, U2 SPX3819-3.3

Commit message: motor peripherals
Parts:
- added C6: 0.1uF, Capacitor_SMD:C_0805_2012Metric, symbol Device:C_Small
- added D2: 50V1A, Diode_SMD:D_0805_2012Metric, symbol Device:D_Small
- added Q3: NPN30V1A, Package_TO_SOT_SMD:SOT-23, symbol Transistor_BJT:2N2219
- added R5: 1kΩ, Resistor_SMD:R_0805_2012Metric, symbol Device:R_Small
Connections:
- net +3V3: now also TP15.1, C6.1, D2.1 (K)
- net GND: now also Q3.1 (E); no longer TP16.1
- net VIB: now also R5.2; no longer TP15.1
- new net: C6.2, D2.2 (A), Q3.3 (C), TP16.1
- new net: Q3.2 (B), R5.1
Other:
- moved on the sheet: M1, TP15, TP16

Commit message: hanging changes
Parts:
- D2: symbol Device:D_Small -> Device:D_Schottky_Small
Changed lines of the file:
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@@
     (pin "1")
   )
-  (symbol (lib_id "Device:D_Small") (at 153.035 73.025 270) (unit 1)
+  (symbol (lib_id "Device:D_Schottky_Small") (at 153.035 73.025 270) (unit 1)
     (in_bom yes) (on_board yes)
     (property "Reference" "D2" (id 0) (at 148.59 73.025 90)

Commit message: pcb update
Parts:
- removed TP10, TP11, TP9: TestPoint_Alt, cap_pads:CAPPADS_7.6x11.6_Chevron_2, symbol Connector:TestPoint_Alt
- removed TP12: TestPoint_Alt, cap_pads:CAPPADS_7.6x11.6_Chevron_3, symbol Connector:TestPoint_Alt
- TP1: footprint cap_pads:CAPPADS_7.6x11.6_Chevron_1 -> cap_pads:CAPPAD_11.4x11.6_1
- TP2, TP3, TP4, TP5, TP6, TP7: footprint cap_pads:CAPPADS_7.6x11.6_Chevron_2 -> cap_pads:CAPPAD_11.4x11.6_2
- TP8: footprint cap_pads:CAPPADS_7.6x11.6_Chevron_2 -> cap_pads:CAPPAD_11.4x11.6_3
Connections:
- no-connect marks 0 -> 4
Changed lines of the file:
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@@
   (junction (at 51.435 41.275) (diameter 0) (color 0 0 0 0)
   )
+  (no_connect (at 125.73 66.675))
+  (no_connect (at 125.73 69.215))
+  (no_connect (at 125.73 71.755))
+  (no_connect (at 126.365 74.295))
   (wire (pts (xy 151.765 83.185) (xy 153.035 83.185))
     (stroke (width 0) (type default) (color 0 0 0 0))
@@
     (stroke (width 0) (type default) (color 0 0 0 0))
   )
-  (wire (pts (xy 125.73 66.675) (xy 127 66.675))
-    (stroke (width 0) (type default) (color 0 0 0 0))
-  )
   (wire (pts (xy 146.685 46.355) (xy 146.685 54.61))
     (stroke (width 0) (type default) (color 0 0 0 0))
   )
-  (wire (pts (xy 125.73 74.295) (xy 127 74.295))
-    (stroke (width 0) (type default) (color 0 0 0 0))
-  )
   (wire (pts (xy 160.655 48.895) (xy 161.925 48.895))
     (stroke (width 0) (type default) (color 0 0 0 0))
@@
     (stroke (width 0) (type default) (color 0 0 0 0))
   )
-  (wire (pts (xy 125.73 71.755) (xy 127 71.755))
-    (stroke (width 0) (type default) (color 0 0 0 0))
-  )
   (wire (pts (xy 35.56 52.705) (xy 35.56 51.435))
     (stroke (width 0) (type default) (color 0 0 0 0))
@@
   )
   (wire (pts (xy 99.06 71.755) (xy 99.06 73.025))
-    (stroke (width 0) (type default) (color 0 0 0 0))
-  )
-  (wire (pts (xy 125.73 69.215) (xy 127 69.215))
     (stroke (width 0) (type default) (color 0 0 0 0))
   )
@@
     (pin "5")
   )
-  (symbol (lib_id "Connector:TestPoint_Alt") (at 127 74.295 270) (unit 1)
-    (in_bom yes) (on_board yes)
-    (property "Reference" "TP12" (id 0) (at 131.445 74.295 90)
-      (effects (font (size 1.27 1.27)) (justify left))
-    )
-    (property "Value" "TestPoint_Alt" (id 1) (at 131.445 74.93 90)
-      (effects (font (size 1.27 1.27)) (justify left) hide)
-    )
-    (property "Footprint" "cap_pads:CAPPADS_7.6x11.6_Chevron_3" (id 2) (at 127 79.375 0)
-      (effects (font (size 1.27 1.27)) hide)
-    )
-    (property "Datasheet" "~" (id 3) (at 127 79.375 0)
-      (effects (font (size 1.27 1.27)) hide)
-    )
-    (pin "1")
-  )
   (symbol (lib_id "Mechanical:MountingHole") (at 38.735 71.12 0) (unit 1)
     (in_bom yes) (on_board yes) (fields_autoplaced)
@@
     )
     (property "Datasheet" "" (id 3) (at 22.225 52.705 0)
-      (effects (font (size 1.27 1.27)) hide)
-    )
-    (pin "1")
-  )
-  (symbol (lib_id "Connector:TestPoint_Alt") (at 127 66.675 270) (unit 1)
-    (in_bom yes) (on_board yes)
-    (property "Reference" "TP9" (id 0) (at 131.445 66.675 90)
-      (effects (font (size 1.27 1.27)) (justify left))
-    )
-    (property "Value" "TestPoint_Alt" (id 1) (at 131.445 67.31 90)
-      (effects (font (size 1.27 1.27)) (justify left) hide)
-    )
-    (property "Footprint" "cap_pads:CAPPADS_7.6x11.6_Chevron_2" (id 2) (at 127 71.755 0)
-      (effects (font (size 1.27 1.27)) hide)
-    )
-    (property "Datasheet" "~" (id 3) (at 127 71.755 0)
       (effects (font (size 1.27 1.27)) hide)
     )
@@
       (effects (font (size 1.27 1.27)) (justify left) hide)
     )
-    (property "Footprint" "cap_pads:CAPPADS_7.6x11.6_Chevron_2" (id 2) (at 127 69.215 0)
+    (property "Footprint" "cap_pads:CAPPAD_11.4x11.6_3" (id 2) (at 127 69.215 0)
       (effects (font (size 1.27 1.27)) hide)
     )
     (property "Datasheet" "~" (id 3) (at 127 69.215 0)
-      (effects (font (size 1.27 1.27)) hide)
-    )
-    (pin "1")
-  )
-  (symbol (lib_id "Connector:TestPoint_Alt") (at 127 71.755 270) (unit 1)
-    (in_bom yes) (on_board yes)
-    (property "Reference" "TP11" (id 0) (at 131.445 71.755 90)
-      (effects (font (size 1.27 1.27)) (justify left))
-    )
-    (property "Value" "TestPoint_Alt" (id 1) (at 131.445 72.39 90)
-      (effects (font (size 1.27 1.27)) (justify left) hide)
-    )
-    (property "Footprint" "cap_pads:CAPPADS_7.6x11.6_Chevron_2" (id 2) (at 127 76.835 0)
-      (effects (font (size 1.27 1.27)) hide)
-    )
-    (property "Datasheet" "~" (id 3) (at 127 76.835 0)
       (effects (font (size 1.27 1.27)) hide)
     )
@@
       (effects (font (size 1.27 1.27)) (justify left) hide)
     )
-    (property "Footprint" "cap_pads:CAPPADS_7.6x11.6_Chevron_2" (id 2) (at 127 56.515 0)
+    (property "Footprint" "cap_pads:CAPPAD_11.4x11.6_2" (id 2) (at 127 56.515 0)
       (effects (font (size 1.27 1.27)) hide)
     )
@@
       (effects (font (size 1.27 1.27)) (justify left) hide)
     )
-    (property "Footprint" "cap_pads:CAPPADS_7.6x11.6_Chevron_2" (id 2) (at 127 61.595 0)
+    (property "Footprint" "cap_pads:CAPPAD_11.4x11.6_2" (id 2) (at 127 61.595 0)
       (effects (font (size 1.27 1.27)) hide)
     )
@@
       (effects (font (size 1.27 1.27)) (justify left) hide)
     )
-    (property "Footprint" "cap_pads:CAPPADS_7.6x11.6_Chevron_2" (id 2) (at 127 53.975 0)
+    (property "Footprint" "cap_pads:CAPPAD_11.4x11.6_2" (id 2) (at 127 53.975 0)
       (effects (font (size 1.27 1.27)) hide)
     )
@@
       (effects (font (size 1.27 1.27)) (justify left) hide)
     )
-    (property "Footprint" "cap_pads:CAPPADS_7.6x11.6_Chevron_2" (id 2) (at 127 66.675 0)
+    (property "Footprint" "cap_pads:CAPPAD_11.4x11.6_2" (id 2) (at 127 66.675 0)
       (effects (font (size 1.27 1.27)) hide)
     )
@@
       (effects (font (size 1.27 1.27)) (justify left) hide)
     )
-    (property "Footprint" "cap_pads:CAPPADS_7.6x11.6_Chevron_2" (id 2) (at 127 59.055 0)
+    (property "Footprint" "cap_pads:CAPPAD_11.4x11.6_2" (id 2) (at 127 59.055 0)
       (effects (font (size 1.27 1.27)) hide)
     )
@@
       (effects (font (size 1.27 1.27)) (justify left) hide)
     )
-    (property "Footprint" "cap_pads:CAPPADS_7.6x11.6_Chevron_1" (id 2) (at 127 51.435 0)
+    (property "Footprint" "cap_pads:CAPPAD_11.4x11.6_1" (id 2) (at 127 51.435 0)
       (effects (font (size 1.27 1.27)) hide)
     )
@@
       (effects (font (size 1.27 1.27)) (justify left) hide)
     )
-    (property "Footprint" "cap_pads:CAPPADS_7.6x11.6_Chevron_2" (id 2) (at 127 64.135 0)
+    (property "Footprint" "cap_pads:CAPPAD_11.4x11.6_2" (id 2) (at 127 64.135 0)
       (effects (font (size 1.27 1.27)) hide)
     )
@@
     (pin "1")
   )
-  (symbol (lib_id "Connector:TestPoint_Alt") (at 127 69.215 270) (unit 1)
-    (in_bom yes) (on_board yes)
-    (property "Reference" "TP10" (id 0) (at 131.445 69.215 90)
-      (effects (font (size 1.27 1.27)) (justify left))
-    )
-    (property "Value" "TestPoint_Alt" (id 1) (at 131.445 69.85 90)
-      (effects (font (size 1.27 1.27)) (justify left) hide)
-    )
-    (property "Footprint" "cap_pads:CAPPADS_7.6x11.6_Chevron_2" (id 2) (at 127 74.295 0)
-      (effects (font (size 1.27 1.27)) hide)
-    )
-    (property "Datasheet" "~" (id 3) (at 127 74.295 0)
-      (effects (font (size 1.27 1.27)) hide)
-    )
-    (pin "1")
-  )
   (symbol (lib_id "power:+3V3") (at 58.42 40.005 0) (unit 1)
     (in_bom yes) (on_board yes)
@@
     )
     (path "/ba1958a1-7d76-4e1e-8b73-7c7712e56926"
-      (reference "TP1") (unit 1) (value "TestPoint_Alt") (footprint "cap_pads:CAPPADS_7.6x11.6_Chevron_1")
+      (reference "TP1") (unit 1) (value "TestPoint_Alt") (footprint "cap_pads:CAPPAD_11.4x11.6_1")
     )
     (path "/8b9944d7-de45-4c10-8f23-654b52f4b910"
-      (reference "TP2") (unit 1) (value "TestPoint_Alt") (footprint "cap_pads:CAPPADS_7.6x11.6_Chevron_2")
+      (reference "TP2") (unit 1) (value "TestPoint_Alt") (footprint "cap_pads:CAPPAD_11.4x11.6_2")
     )
     (path "/619d42dc-7a77-4d03-bcdd-97078c405047"
-      (reference "TP3") (unit 1) (value "TestPoint_Alt") (footprint "cap_pads:CAPPADS_7.6x11.6_Chevron_2")
+      (reference "TP3") (unit 1) (value "TestPoint_Alt") (footprint "cap_pads:CAPPAD_11.4x11.6_2")
     )
     (path "/b829908f-cd58-4d41-823c-96c17337397b"
-      (reference "TP4") (unit 1) (value "TestPoint_Alt") (footprint "cap_pads:CAPPADS_7.6x11.6_Chevron_2")
+      (reference "TP4") (unit 1) (value "TestPoint_Alt") (footprint "cap_pads:CAPPAD_11.4x11.6_2")
     )
     (path "/625a82e9-f251-4d4b-85a0-987cbbd608cd"
-      (reference "TP5") (unit 1) (value "TestPoint_Alt") (footprint "cap_pads:CAPPADS_7.6x11.6_Chevron_2")
+      (reference "TP5") (unit 1) (value "TestPoint_Alt") (footprint "cap_pads:CAPPAD_11.4x11.6_2")
     )
     (path "/bc614aae-bf8a-4524-b8fb-f2986c6a385f"
-      (reference "TP6") (unit 1) (value "TestPoint_Alt") (footprint "cap_pads:CAPPADS_7.6x11.6_Chevron_2")
+      (reference "TP6") (unit 1) (value "TestPoint_Alt") (footprint "cap_pads:CAPPAD_11.4x11.6_2")
     )
     (path "/b13c650d-d345-428a-ba03-fd5871ca5c98"
-      (reference "TP7") (unit 1) (value "TestPoint_Alt") (footprint "cap_pads:CAPPADS_7.6x11.6_Chevron_2")
+      (reference "TP7") (unit 1) (value "TestPoint_Alt") (footprint "cap_pads:CAPPAD_11.4x11.6_2")
     )
     (path "/4e184203-7c1c-4b52-a73a-be217f4bb796"
-      (reference "TP8") (unit 1) (value "TestPoint_Alt") (footprint "cap_pads:CAPPADS_7.6x11.6_Chevron_2")
-    )
-    (path "/39942e6b-3cc0-4ee7-8c07-44ca728f58d6"
-      (reference "TP9") (unit 1) (value "TestPoint_Alt") (footprint "cap_pads:CAPPADS_7.6x11.6_Chevron_2")
-    )
-    (path "/f030bf22-0011-4c17-a015-6e34a85a327f"
-      (reference "TP10") (unit 1) (value "TestPoint_Alt") (footprint "cap_pads:CAPPADS_7.6x11.6_Chevron_2")
-    )
-    (path "/5200f4f7-8155-455b-8d82-55039fa33a17"
-      (reference "TP11") (unit 1) (value "TestPoint_Alt") (footprint "cap_pads:CAPPADS_7.6x11.6_Chevron_2")
-    )
-    (path "/1db37ab1-6540-4715-a5f1-8f515d3788c5"
-      (reference "TP12") (unit 1) (value "TestPoint_Alt") (footprint "cap_pads:CAPPADS_7.6x11.6_Chevron_3")
+      (reference "TP8") (unit 1) (value "TestPoint_Alt") (footprint "cap_pads:CAPPAD_11.4x11.6_3")
     )
     (path "/fd00f671-a567-4561-b2a9-081b479a0835"
