File: pcb/touchpad_daughterboard/cap64pcb.kicad_pcb (KiCad board)
At the start: 2 copper layers, 91.6 x 12 mm, 35 parts, among them J1 SM04B_SURS_TF, M1 Coin_Motor, Q1 BSS138, Q2 BSS138, U1 MPR121QR2, U2 SPX3819-3.3

Commit message: remove JLCJLCJLCJLC
Other:
- board text removed: "JLCJLCJLCJLC"
Changed lines of the file:
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@@
     (effects (font (size 1 1) (thickness 0.2)) (justify left mirror))
-  )
-  (gr_text "JLCJLCJLCJLC" (at 80 46.6) (layer "B.SilkS")
-    (effects (font (size 0.85 0.85) (thickness 0.2)) (justify mirror))
   )
   (gr_text "JST-\nSURS" (at 115.5 41.7 90) (layer "B.SilkS")

Commit message: touchpad silk raster
Parts:
- added G***: LOGO, logo:cap_back_silkraster, B.Cu at (80.0, 45.0)
Other:
- board text removed: "0x5[abcd]"
- board text removed: "64"
- board text removed: "JST- SURS"
- board text removed: "Vibin'"
- board text removed: "beady"
- board text removed: "biddle"
- board text removed: "cap"
- board text removed: "gnd"
- board text removed: "scl"
- board text removed: "sda"
- board text removed: "vcc"
- board text removed: "vib"
