File: pcb/motherboard/bd64pcb.kicad_sch (KiCad schematic)
At the start: 224 parts, among them J1 SM04B-SRSS-TB, J2 SM05B-SURS-TF, J3 SM05B-SURS-TF, SW1 SW_Push, U1 ATmega32U4-MU, U2 IS31FL3733-QF, Y1 16MHz

Commit message: mht symbols & footprint
Parts:
- L1, L10, L11, L12, L13, L14, L15, L16, L17, L18, L19, L2, L20, L21, L22, L23, L24, L25, L26, L27, L28, L29, L3, L30, L31, L32, L33, L34, L35, L36, L37, L38, L39, L4, L40, L41, L42, L43, L44, L45, L46, L47, L48, L49, L5, L50, L51, L52, L53, L54, L55, L56, L57, L58, L59, L6, L60, L61, L62, L63, L64, L7, L8, L9: value QBLP677R-RGB -> MHT151RGBCT; footprint QBLP677R-RGB:RGB-REVERSE_MOUNT -> MHT151RGBCT:MHT151RGBCT_REVERSE_MOUNT; symbol QBLP677R-RGB:QBLP677R-RGB -> MHT151RGBCT:MHT151RGBCT
Connections:
- net SW1: now also L1.3, L10.3, L11.3, L12.3, L13.3, L14.3, L15.3, L16.3, L2.3, L3.3, L4.3, L5.3, L6.3, L7.3, L8.3, L9.3; no longer L1.2, L10.2, L11.2, L12.2, L13.2, L14.2, L15.2, L16.2, L2.2, L3.2, L4.2, L5.2, L6.2, L7.2, L8.2, L9.2
- net SW10: now also L49.3, L50.3, L51.3, L52.3, L53.3, L54.3, L55.3, L56.3, L57.3, L58.3, L59.3, L60.3, L61.3, L62.3, L63.3, L64.3; no longer L49.2, L50.2, L51.2, L52.2, L53.2, L54.2, L55.2, L56.2, L57.2, L58.2, L59.2, L60.2, L61.2, L62.2, L63.2, L64.2
- net SW11: now also L49.4, L50.4, L51.4, L52.4, L53.4, L54.4, L55.4, L56.4, L57.4, L58.4, L59.4, L60.4, L61.4, L62.4, L63.4, L64.4; no longer L49.3, L50.3, L51.3, L52.3, L53.3, L54.3, L55.3, L56.3, L57.3, L58.3, L59.3, L60.3, L61.3, L62.3, L63.3, L64.3
- net SW12: now also L49.2, L50.2, L51.2, L52.2, L53.2, L54.2, L55.2, L56.2, L57.2, L58.2, L59.2, L60.2, L61.2, L62.2, L63.2, L64.2; no longer L49.1, L50.1, L51.1, L52.1, L53.1, L54.1, L55.1, L56.1, L57.1, L58.1, L59.1, L60.1, L61.1, L62.1, L63.1, L64.1
- net SW2: now also L1.4, L10.4, L11.4, L12.4, L13.4, L14.4, L15.4, L16.4, L2.4, L3.4, L4.4, L5.4, L6.4, L7.4, L8.4, L9.4; no longer L1.3, L10.3, L11.3, L12.3, L13.3, L14.3, L15.3, L16.3, L2.3, L3.3, L4.3, L5.3, L6.3, L7.3, L8.3, L9.3
- net SW3: now also L1.2, L10.2, L11.2, L12.2, L13.2, L14.2, L15.2, L16.2, L2.2, L3.2, L4.2, L5.2, L6.2, L7.2, L8.2, L9.2; no longer L1.1, L10.1, L11.1, L12.1, L13.1, L14.1, L15.1, L16.1, L2.1, L3.1, L4.1, L5.1, L6.1, L7.1, L8.1, L9.1
- net SW4: now also L17.3, L18.3, L19.3, L20.3, L21.3, L22.3, L23.3, L24.3, L25.3, L26.3, L27.3, L28.3, L29.3, L30.3, L31.3, L32.3; no longer L17.2, L18.2, L19.2, L20.2, L21.2, L22.2, L23.2, L24.2, L25.2, L26.2, L27.2, L28.2, L29.2, L30.2, L31.2, L32.2
- net SW5: now also L17.4, L18.4, L19.4, L20.4, L21.4, L22.4, L23.4, L24.4, L25.4, L26.4, L27.4, L28.4, L29.4, L30.4, L31.4, L32.4; no longer L17.3, L18.3, L19.3, L20.3, L21.3, L22.3, L23.3, L24.3, L25.3, L26.3, L27.3, L28.3, L29.3, L30.3, L31.3, L32.3
- net SW6: now also L17.2, L18.2, L19.2, L20.2, L21.2, L22.2, L23.2, L24.2, L25.2, L26.2, L27.2, L28.2, L29.2, L30.2, L31.2, L32.2; no longer L17.1, L18.1, L19.1, L20.1, L21.1, L22.1, L23.1, L24.1, L25.1, L26.1, L27.1, L28.1, L29.1, L30.1, L31.1, L32.1
- net SW7: now also L33.3, L34.3, L35.3, L36.3, L37.3, L38.3, L39.3, L40.3, L41.3, L42.3, L43.3, L44.3, L45.3, L46.3, L47.3, L48.3; no longer L33.2, L34.2, L35.2, L36.2, L37.2, L38.2, L39.2, L40.2, L41.2, L42.2, L43.2, L44.2, L45.2, L46.2, L47.2, L48.2
- net SW8: now also L33.4, L34.4, L35.4, L36.4, L37.4, L38.4, L39.4, L40.4, L41.4, L42.4, L43.4, L44.4, L45.4, L46.4, L47.4, L48.4; no longer L33.3, L34.3, L35.3, L36.3, L37.3, L38.3, L39.3, L40.3, L41.3, L42.3, L43.3, L44.3, L45.3, L46.3, L47.3, L48.3
- net SW9: now also L33.2, L34.2, L35.2, L36.2, L37.2, L38.2, L39.2, L40.2, L41.2, L42.2, L43.2, L44.2, L45.2, L46.2, L47.2, L48.2; no longer L33.1, L34.1, L35.1, L36.1, L37.1, L38.1, L39.1, L40.1, L41.1, L42.1, L43.1, L44.1, L45.1, L46.1, L47.1, L48.1
